Commit message: simulation fixes

File: assets/creatures/1-spherical_hopper.urdf (robot description, URDF)
Before this commit: robot spherical_hopper, 2 links, 1 joints
Joints:
- joint spine_joint: limit lower=-1.57 -1.57 -1.57 upper=1.57 1.57 1.57 effort=20 velocity=10 -> (none)

Commit message: fixed default motor control blocking spherical joint movement, various other creature and simulation fixes

File: assets/creatures/1-spherical_hopper.urdf (robot description, URDF)
Before this commit: robot 1-spherical_hopper, 2 links, 1 joints
Joints:
- joint spine_joint: limit (none) -> effort=10000 velocity=100

File: assets/creatures/2-spherical_2-revolute_two-arm-biped.urdf (robot description, URDF)
Before this commit: robot 2-spherical_2-revolute_two-arm-biped, 5 links, 4 joints
Joints:
- joint hip_left: limit lower=-0.785 upper=0.785 effort=12 velocity=6 -> effort=10000 velocity=100
- joint hip_right: limit lower=-0.785 upper=0.785 effort=12 velocity=6 -> effort=10000 velocity=100
- joint shoulder_left: limit lower=-1.57 -1.57 -1.57 upper=1.57 1.57 1.57 effort=10 velocity=5 -> effort=10000 velocity=100
- joint shoulder_right: limit lower=-1.57 -1.57 -1.57 upper=1.57 1.57 1.57 effort=10 velocity=5 -> effort=10000 velocity=100

File: assets/creatures/4-spherical_4-revolute_spider-bot.urdf (robot description, URDF)
Before this commit: robot 4-spherical_4-revolute_spider-bot, 9 links, 8 joints
Links:
- link body_core: mass 3 -> 1.5
- link hip_bl_link: mass 0.1 -> 0.3
- link hip_br_link: mass 0.1 -> 0.3
- link hip_fl_link: mass 0.1 -> 0.3
- link hip_fr_link: mass 0.1 -> 0.3
- link knee_bl_link: mass 0.1 -> 0.3
- link knee_br_link: mass 0.1 -> 0.3
- link knee_fl_link: mass 0.1 -> 0.3
- link knee_fr_link: mass 0.1 -> 0.3
Joints:
- joint hip_bl: limit lower=-1.0 -1.0 -1.0 upper=1.0 1.0 1.0 effort=10 velocity=5 -> effort=10000 velocity=100
- joint hip_br: limit lower=-1.0 -1.0 -1.0 upper=1.0 1.0 1.0 effort=10 velocity=5 -> effort=10000 velocity=100
- joint hip_fl: limit lower=-1.0 -1.0 -1.0 upper=1.0 1.0 1.0 effort=10 velocity=5 -> effort=10000 velocity=100
- joint hip_fr: limit lower=-1.0 -1.0 -1.0 upper=1.0 1.0 1.0 effort=10 velocity=5 -> effort=10000 velocity=100
- joint knee_bl: limit lower=-1.57 upper=0 effort=8 velocity=4 -> effort=10000 velocity=100
- joint knee_br: limit lower=-1.57 upper=0 effort=8 velocity=4 -> effort=10000 velocity=100
- joint knee_fl: limit lower=-1.57 upper=0 effort=8 velocity=4 -> effort=10000 velocity=100
- joint knee_fr: limit lower=-1.57 upper=0 effort=8 velocity=4 -> effort=10000 velocity=100

File: assets/creatures/4-spherical_quadruped.urdf (robot description, URDF)
Before this commit: robot 5-spherical_quadruped, 5 links, 4 joints
Links:
- link leg_bl: geometry collision cylinder length=0.02 radius=0.1; visual cylinder length=0.02 radius=0.1
- link leg_br: geometry collision cylinder length=0.02 radius=0.1; visual cylinder length=0.02 radius=0.1
- link leg_fl: geometry collision cylinder length=0.02 radius=0.1; visual cylinder length=0.02 radius=0.1
- link leg_fr: geometry collision cylinder length=0.02 radius=0.1; visual cylinder length=0.02 radius=0.1
Joints:
- joint hip_bl: limit lower=-1.0 -1.0 -1.0 upper=1.0 1.0 1.0 effort=15 velocity=8 -> effort=10000 velocity=100
- joint hip_br: limit lower=-1.0 -1.0 -1.0 upper=1.0 1.0 1.0 effort=15 velocity=8 -> effort=10000 velocity=100
- joint hip_fl: limit lower=-1.0 -1.0 -1.0 upper=1.0 1.0 1.0 effort=15 velocity=8 -> effort=10000 velocity=100
- joint hip_fr: limit lower=-1.0 -1.0 -1.0 upper=1.0 1.0 1.0 effort=15 velocity=8 -> effort=10000 velocity=100

File: assets/creatures/6-revolute_biped.urdf (robot description, URDF)
Before this commit: robot 6-revolute_biped, 7 links, 6 joints
Joints:
- joint left_ankle: limit lower=-0.785 upper=0.785 effort=100 velocity=10 -> effort=10000 velocity=100
- joint left_hip: limit lower=-1.57 upper=1.57 effort=100 velocity=10 -> effort=10000 velocity=100
- joint left_knee: limit lower=0 upper=1.57 effort=100 velocity=10 -> effort=10000 velocity=100
- joint right_ankle: limit lower=-0.785 upper=0.785 effort=100 velocity=10 -> effort=10000 velocity=100
- joint right_hip: limit lower=-1.57 upper=1.57 effort=100 velocity=10 -> effort=10000 velocity=100
- joint right_knee: limit lower=0 upper=1.57 effort=100 velocity=10 -> effort=10000 velocity=100

Commit message: added fitness function and run conditions that punish falling over

File: assets/creatures/1-spherical_hopper.urdf (robot description, URDF)
Before this commit: robot 1-spherical_hopper, 2 links, 1 joints
Links:
- removed link upper_body
- added link leg, mass 1.5; collision sphere radius=0.2; visual sphere radius=0.2
- link base_link: mass 1.5 -> 1.0; geometry collision sphere radius=0.15; visual sphere radius=0.15
Joints:
- removed joint spine_joint
- added joint leg_joint: type spherical, parent base_link, child leg, origin xyz=0 0 -0.35 rpy=0 0 0, limit effort=10000 velocity=100

Commit message: fixed negative species sizes

File: assets/creatures/1-spherical_hopper.urdf (robot description, URDF)
Before this commit: robot 1-spherical_hopper, 2 links, 1 joints
Joints:
- joint leg_joint: axis (none) -> 1 0 0

Commit message: corrected 3d model's parameters, fixed model clipping into the ground

File: assets/creatures/1-spherical_hopper.urdf (robot description, URDF)
Before this commit: robot 1-spherical_hopper, 2 links, 1 joints
Joints:
- joint leg_joint: axis 1 0 0 -> (none); limit effort=10000 velocity=100 -> effort=200 velocity=20

File: assets/creatures/2-spherical_2-revolute_two-arm-biped.urdf (robot description, URDF)
Before this commit: robot 2-spherical_2-revolute_two-arm-biped, 5 links, 4 joints
Joints:
- joint hip_left: limit effort=10000 velocity=100 -> lower=-0.8 upper=0.8 effort=200 velocity=20
- joint hip_right: limit effort=10000 velocity=100 -> lower=-0.8 upper=0.8 effort=200 velocity=20
- joint shoulder_left: limit effort=10000 velocity=100 -> effort=100 velocity=20
- joint shoulder_right: limit effort=10000 velocity=100 -> effort=100 velocity=20

File: assets/creatures/4-spherical_4-revolute_spider-bot.urdf (robot description, URDF)
Before this commit: robot 4-spherical_4-revolute_spider-bot, 9 links, 8 joints
Joints:
- joint hip_bl: limit effort=10000 velocity=100 -> effort=150 velocity=20
- joint hip_br: limit effort=10000 velocity=100 -> effort=150 velocity=20
- joint hip_fl: limit effort=10000 velocity=100 -> effort=150 velocity=20
- joint hip_fr: limit effort=10000 velocity=100 -> effort=150 velocity=20
- joint knee_bl: limit effort=10000 velocity=100 -> lower=-0.1 upper=2.5 effort=150 velocity=20
- joint knee_br: limit effort=10000 velocity=100 -> lower=-0.1 upper=2.5 effort=150 velocity=20
- joint knee_fl: limit effort=10000 velocity=100 -> lower=-0.1 upper=2.5 effort=150 velocity=20
- joint knee_fr: limit effort=10000 velocity=100 -> lower=-0.1 upper=2.5 effort=150 velocity=20

File: assets/creatures/4-spherical_quadruped.urdf (robot description, URDF)
Before this commit: robot 4-spherical_quadruped, 5 links, 4 joints
Joints:
- joint hip_bl: limit effort=10000 velocity=100 -> effort=150 velocity=20
- joint hip_br: limit effort=10000 velocity=100 -> effort=150 velocity=20
- joint hip_fl: limit effort=10000 velocity=100 -> effort=150 velocity=20
- joint hip_fr: limit effort=10000 velocity=100 -> effort=150 velocity=20

File: assets/creatures/6-revolute_biped.urdf (robot description, URDF)
Before this commit: robot 6-revolute_biped, 7 links, 6 joints
Joints:
- joint left_ankle: limit effort=10000 velocity=100 -> lower=-0.4 upper=0.4 effort=100 velocity=20
- joint left_hip: limit effort=10000 velocity=100 -> lower=-0.8 upper=0.8 effort=200 velocity=20
- joint left_knee: limit effort=10000 velocity=100 -> lower=0.0 upper=2.5 effort=200 velocity=20
- joint right_ankle: limit effort=10000 velocity=100 -> lower=-0.4 upper=0.4 effort=100 velocity=20
- joint right_hip: limit effort=10000 velocity=100 -> lower=-0.8 upper=0.8 effort=200 velocity=20
- joint right_knee: limit effort=10000 velocity=100 -> lower=0.0 upper=2.5 effort=200 velocity=20

Commit message: features: added saving global best individual every generation fixes: made paths in params relative for better retrievability, fixed pybullet warnings

File: assets/creatures/1-spherical_hopper.urdf (robot description, URDF)
Before this commit: robot 1-spherical_hopper, 2 links, 1 joints
Joints:
- joint leg_joint: axis (none) -> 1 0 0

File: assets/creatures/2-spherical_2-revolute_two-arm-biped.urdf (robot description, URDF)
Before this commit: robot 2-spherical_2-revolute_two-arm-biped, 5 links, 4 joints
Joints:
- joint shoulder_left: axis (none) -> 1 0 0
- joint shoulder_right: axis (none) -> 1 0 0

File: assets/creatures/4-spherical_quadruped.urdf (robot description, URDF)
Before this commit: robot 4-spherical_quadruped, 5 links, 4 joints
Joints:
- joint hip_bl: axis (none) -> 1 0 0
- joint hip_br: axis (none) -> 1 0 0
- joint hip_fl: axis (none) -> 1 0 0
- joint hip_fr: axis (none) -> 1 0 0

Commit message: fixed creature joint parameters, fixed docstrings

File: assets/creatures/1-spherical_hopper.urdf (robot description, URDF)
Before this commit: robot 1-spherical_hopper, 2 links, 1 joints
Joints:
- joint leg_joint: axis 1 0 0 -> 0 0 1; limit effort=200 velocity=20 -> effort=50 velocity=5.0

File: assets/creatures/2-spherical_2-revolute_two-arm-biped.urdf (robot description, URDF)
Before this commit: robot 2-spherical_2-revolute_two-arm-biped, 5 links, 4 joints
Joints:
- joint hip_left: limit lower=-0.8 upper=0.8 effort=200 velocity=20 -> lower=-0.8 upper=0.8 effort=30 velocity=5.0
- joint hip_right: limit lower=-0.8 upper=0.8 effort=200 velocity=20 -> lower=-0.8 upper=0.8 effort=30 velocity=5.0
- joint shoulder_left: axis 1 0 0 -> 0 0 1; limit effort=100 velocity=20 -> effort=10 velocity=5.0
- joint shoulder_right: axis 1 0 0 -> 0 0 1; limit effort=100 velocity=20 -> effort=10 velocity=5.0

File: assets/creatures/4-spherical_4-revolute_spider-bot.urdf (robot description, URDF)
Before this commit: robot 4-spherical_4-revolute_spider-bot, 9 links, 8 joints
Joints:
- joint hip_bl: limit effort=150 velocity=20 -> effort=50 velocity=5.0
- joint hip_br: limit effort=150 velocity=20 -> effort=50 velocity=5.0
- joint hip_fl: limit effort=150 velocity=20 -> effort=50 velocity=5.0
- joint hip_fr: limit effort=150 velocity=20 -> effort=50 velocity=5.0
- joint knee_bl: limit lower=-0.1 upper=2.5 effort=150 velocity=20 -> lower=-0.1 upper=2.5 effort=40 velocity=5.0
- joint knee_br: limit lower=-0.1 upper=2.5 effort=150 velocity=20 -> lower=-0.1 upper=2.5 effort=40 velocity=5.0
- joint knee_fl: limit lower=-0.1 upper=2.5 effort=150 velocity=20 -> lower=-0.1 upper=2.5 effort=40 velocity=5.0
- joint knee_fr: limit lower=-0.1 upper=2.5 effort=150 velocity=20 -> lower=-0.1 upper=2.5 effort=40 velocity=5.0

File: assets/creatures/4-spherical_quadruped.urdf (robot description, URDF)
Before this commit: robot 4-spherical_quadruped, 5 links, 4 joints
Joints:
- joint hip_bl: axis 1 0 0 -> 0 0 1; limit effort=150 velocity=20 -> effort=50 velocity=5.0
- joint hip_br: axis 1 0 0 -> 0 0 1; limit effort=150 velocity=20 -> effort=50 velocity=5.0
- joint hip_fl: axis 1 0 0 -> 0 0 1; limit effort=150 velocity=20 -> effort=50 velocity=5.0
- joint hip_fr: axis 1 0 0 -> 0 0 1; limit effort=150 velocity=20 -> effort=50 velocity=5.0

File: assets/creatures/6-revolute_biped.urdf (robot description, URDF)
Before this commit: robot 6-revolute_biped, 7 links, 6 joints
Joints:
- joint left_ankle: limit lower=-0.4 upper=0.4 effort=100 velocity=20 -> lower=-0.4 upper=0.4 effort=40 velocity=5.0
- joint right_ankle: limit lower=-0.4 upper=0.4 effort=100 velocity=20 -> lower=-0.4 upper=0.4 effort=40 velocity=5.0

Commit message: reverted models' changes

File: assets/creatures/1-spherical_hopper.urdf (robot description, URDF)
Before this commit: robot 1-spherical_hopper, 2 links, 1 joints
Joints:
- joint leg_joint: axis 0 0 1 -> 1 0 0; limit effort=50 velocity=5.0 -> effort=200 velocity=20

File: assets/creatures/2-spherical_2-revolute_two-arm-biped.urdf (robot description, URDF)
Before this commit: robot 2-spherical_2-revolute_two-arm-biped, 5 links, 4 joints
Joints:
- joint hip_left: limit lower=-0.8 upper=0.8 effort=30 velocity=5.0 -> lower=-0.8 upper=0.8 effort=200 velocity=20
- joint hip_right: limit lower=-0.8 upper=0.8 effort=30 velocity=5.0 -> lower=-0.8 upper=0.8 effort=200 velocity=20
- joint shoulder_left: axis 0 0 1 -> 1 0 0; limit effort=10 velocity=5.0 -> effort=100 velocity=20
- joint shoulder_right: axis 0 0 1 -> 1 0 0; limit effort=10 velocity=5.0 -> effort=100 velocity=20

File: assets/creatures/4-spherical_4-revolute_spider-bot.urdf (robot description, URDF)
Before this commit: robot 4-spherical_4-revolute_spider-bot, 9 links, 8 joints
Joints:
- joint hip_bl: limit effort=50 velocity=5.0 -> effort=150 velocity=20
- joint hip_br: limit effort=50 velocity=5.0 -> effort=150 velocity=20
- joint hip_fl: limit effort=50 velocity=5.0 -> effort=150 velocity=20
- joint hip_fr: limit effort=50 velocity=5.0 -> effort=150 velocity=20
- joint knee_bl: limit lower=-0.1 upper=2.5 effort=40 velocity=5.0 -> lower=-0.1 upper=2.5 effort=150 velocity=20
- joint knee_br: limit lower=-0.1 upper=2.5 effort=40 velocity=5.0 -> lower=-0.1 upper=2.5 effort=150 velocity=20
- joint knee_fl: limit lower=-0.1 upper=2.5 effort=40 velocity=5.0 -> lower=-0.1 upper=2.5 effort=150 velocity=20
- joint knee_fr: limit lower=-0.1 upper=2.5 effort=40 velocity=5.0 -> lower=-0.1 upper=2.5 effort=150 velocity=20

File: assets/creatures/4-spherical_quadruped.urdf (robot description, URDF)
Before this commit: robot 4-spherical_quadruped, 5 links, 4 joints
Joints:
- joint hip_bl: axis 0 0 1 -> 1 0 0; limit effort=50 velocity=5.0 -> effort=150 velocity=20
- joint hip_br: axis 0 0 1 -> 1 0 0; limit effort=50 velocity=5.0 -> effort=150 velocity=20
- joint hip_fl: axis 0 0 1 -> 1 0 0; limit effort=50 velocity=5.0 -> effort=150 velocity=20
- joint hip_fr: axis 0 0 1 -> 1 0 0; limit effort=50 velocity=5.0 -> effort=150 velocity=20

File: assets/creatures/6-revolute_biped.urdf (robot description, URDF)
Before this commit: robot 6-revolute_biped, 7 links, 6 joints
Joints:
- joint left_ankle: limit lower=-0.4 upper=0.4 effort=40 velocity=5.0 -> lower=-0.4 upper=0.4 effort=100 velocity=20
- joint right_ankle: limit lower=-0.4 upper=0.4 effort=40 velocity=5.0 -> lower=-0.4 upper=0.4 effort=100 velocity=20

Commit message: fixed simulation not respecting force limits

File: assets/creatures/1-spherical_hopper.urdf (robot description, URDF)
Before this commit: robot 1-spherical_hopper, 2 links, 1 joints
Joints:
- joint leg_joint: axis 1 0 0 -> 0 0 0; limit effort=200 velocity=20 -> effort=60 velocity=6.0

File: assets/creatures/2-spherical_2-revolute_two-arm-biped.urdf (robot description, URDF)
Before this commit: robot 2-spherical_2-revolute_two-arm-biped, 5 links, 4 joints
Joints:
- joint hip_left: limit lower=-0.8 upper=0.8 effort=200 velocity=20 -> lower=-0.8 upper=0.8 effort=50 velocity=6.0
- joint hip_right: limit lower=-0.8 upper=0.8 effort=200 velocity=20 -> lower=-0.8 upper=0.8 effort=50 velocity=6.0
- joint shoulder_left: axis 1 0 0 -> 0 0 0; limit effort=100 velocity=20 -> effort=30 velocity=8.0
- joint shoulder_right: axis 1 0 0 -> 0 0 0; limit effort=100 velocity=20 -> effort=30 velocity=8.0

File: assets/creatures/4-spherical_4-revolute_spider-bot.urdf (robot description, URDF)
Before this commit: robot 4-spherical_4-revolute_spider-bot, 9 links, 8 joints
Links:
- link knee_bl_link: geometry collision cylinder length=0.2 radius=0.03; collision sphere radius=0.03
- link knee_br_link: geometry collision cylinder length=0.2 radius=0.03; collision sphere radius=0.03
- link knee_fl_link: geometry collision cylinder length=0.2 radius=0.03; collision sphere radius=0.03
- link knee_fr_link: geometry collision cylinder length=0.2 radius=0.03; collision sphere radius=0.03
Joints:
- joint hip_bl: limit effort=150 velocity=20 -> effort=80 velocity=6.0
- joint hip_br: limit effort=150 velocity=20 -> effort=80 velocity=6.0
- joint hip_fl: limit effort=150 velocity=20 -> effort=80 velocity=6.0
- joint hip_fr: limit effort=150 velocity=20 -> effort=80 velocity=6.0
- joint knee_bl: limit lower=-0.1 upper=2.5 effort=150 velocity=20 -> lower=-0.1 upper=2.5 effort=60 velocity=8.0
- joint knee_br: limit lower=-0.1 upper=2.5 effort=150 velocity=20 -> lower=-0.1 upper=2.5 effort=60 velocity=8.0
- joint knee_fl: limit lower=-0.1 upper=2.5 effort=150 velocity=20 -> lower=-0.1 upper=2.5 effort=60 velocity=8.0
- joint knee_fr: limit lower=-0.1 upper=2.5 effort=150 velocity=20 -> lower=-0.1 upper=2.5 effort=60 velocity=8.0

File: assets/creatures/4-spherical_quadruped.urdf (robot description, URDF)
Before this commit: robot 4-spherical_quadruped, 5 links, 4 joints
Links:
- link leg_bl: geometry collision cylinder length=0.02 radius=0.1; collision cylinder length=0.24 radius=0.02
- link leg_br: geometry collision cylinder length=0.02 radius=0.1; collision cylinder length=0.24 radius=0.02
- link leg_fl: geometry collision cylinder length=0.02 radius=0.1; collision cylinder length=0.24 radius=0.02
- link leg_fr: geometry collision cylinder length=0.02 radius=0.1; collision cylinder length=0.24 radius=0.02
Joints:
- joint hip_bl: axis 1 0 0 -> 0 0 0; limit effort=150 velocity=20 -> effort=60 velocity=6.0
- joint hip_br: axis 1 0 0 -> 0 0 0; limit effort=150 velocity=20 -> effort=60 velocity=6.0
- joint hip_fl: axis 1 0 0 -> 0 0 0; limit effort=150 velocity=20 -> effort=60 velocity=6.0
- joint hip_fr: axis 1 0 0 -> 0 0 0; limit effort=150 velocity=20 -> effort=60 velocity=6.0

File: assets/creatures/6-revolute_biped.urdf (robot description, URDF)
Before this commit: robot 6-revolute_biped, 7 links, 6 joints
Joints:
- joint left_ankle: limit lower=-0.4 upper=0.4 effort=100 velocity=20 -> lower=-0.4 upper=0.4 effort=40 velocity=4.0
- joint left_hip: limit lower=-0.8 upper=0.8 effort=200 velocity=20 -> lower=-0.8 upper=0.8 effort=150 velocity=6.0
- joint left_knee: limit lower=0.0 upper=2.5 effort=200 velocity=20 -> lower=0.0 upper=2.5 effort=100 velocity=6.0
- joint right_ankle: limit lower=-0.4 upper=0.4 effort=100 velocity=20 -> lower=-0.4 upper=0.4 effort=40 velocity=4.0
- joint right_hip: limit lower=-0.8 upper=0.8 effort=200 velocity=20 -> lower=-0.8 upper=0.8 effort=150 velocity=6.0
- joint right_knee: limit lower=0.0 upper=2.5 effort=200 velocity=20 -> lower=0.0 upper=2.5 effort=100 velocity=6.0
