Commit message: fixed spherical joint movement

File: assets/creatures/2-spherical_2-revolute_two-arm-biped.urdf (robot description, URDF)
Before this commit: robot 2-spherical_2-revolute_two-arm-biped, 5 links, 4 joints
Links:
- link left_arm: mass 0.2 -> 2.0
- link left_leg: mass 0.4 -> 4.0
- link right_arm: mass 0.2 -> 2.0
- link right_leg: mass 0.4 -> 4.0
- link torso: mass 2 -> 20
Joints:
- joint shoulder_left: limit effort=30 velocity=8.0 -> lower=-1.5 upper=1.5 effort=30 velocity=8.0
- joint shoulder_right: limit effort=30 velocity=8.0 -> lower=-1.5 upper=1.5 effort=30 velocity=8.0

File: assets/creatures/4-spherical_4-revolute_spider-bot.urdf (robot description, URDF)
Before this commit: robot 4-spherical_4-revolute_spider-bot, 9 links, 8 joints
Links:
- link body_core: mass 1.5 -> 15.0
- link hip_bl_link: mass 0.3 -> 3.0; geometry collision capsule length=0.18 radius=0.02; visual cylinder length=0.2 radius=0.03
- link hip_br_link: mass 0.3 -> 3.0; geometry collision capsule length=0.18 radius=0.02; visual cylinder length=0.2 radius=0.03
- link hip_fl_link: mass 0.3 -> 3.0; geometry collision capsule length=0.18 radius=0.02; visual cylinder length=0.2 radius=0.03
- link hip_fr_link: mass 0.3 -> 3.0; geometry collision capsule length=0.18 radius=0.02; visual cylinder length=0.2 radius=0.03
- link knee_bl_link: mass 0.3 -> 3.0; geometry collision capsule length=0.18 radius=0.03; collision sphere radius=0.03
- link knee_br_link: mass 0.3 -> 3.0; geometry collision capsule length=0.18 radius=0.03; collision sphere radius=0.03
- link knee_fl_link: mass 0.3 -> 3.0; geometry collision capsule length=0.18 radius=0.03; collision sphere radius=0.03
- link knee_fr_link: mass 0.3 -> 3.0; geometry collision capsule length=0.18 radius=0.03; collision sphere radius=0.03
Joints:
- joint hip_bl: axis (none) -> 0 0 0; limit effort=80 velocity=6.0 -> lower=-0.5 upper=0.5 effort=45 velocity=6.0
- joint hip_br: axis (none) -> 0 0 0; limit effort=80 velocity=6.0 -> lower=-0.5 upper=0.5 effort=45 velocity=6.0
- joint hip_fl: axis (none) -> 0 0 0; limit effort=80 velocity=6.0 -> lower=-0.5 upper=0.5 effort=45 velocity=6.0
- joint hip_fr: axis (none) -> 0 0 0; limit effort=80 velocity=6.0 -> lower=-0.5 upper=0.5 effort=45 velocity=6.0
- joint knee_bl: limit lower=-0.1 upper=2.5 effort=60 velocity=8.0 -> lower=-0.1 upper=2.5 effort=30 velocity=8.0
- joint knee_br: limit lower=-0.1 upper=2.5 effort=60 velocity=8.0 -> lower=-0.1 upper=2.5 effort=30 velocity=8.0
- joint knee_fl: limit lower=-0.1 upper=2.5 effort=60 velocity=8.0 -> lower=-0.1 upper=2.5 effort=30 velocity=8.0
- joint knee_fr: limit lower=-0.1 upper=2.5 effort=60 velocity=8.0 -> lower=-0.1 upper=2.5 effort=30 velocity=8.0

File: assets/creatures/4-spherical_quadruped.urdf (robot description, URDF)
Before this commit: robot 4-spherical_quadruped, 5 links, 4 joints
Links:
- link body: mass 2.5 -> 15.0
- link leg_bl: mass 0.4 -> 5.0
- link leg_br: mass 0.4 -> 5.0
- link leg_fl: mass 0.4 -> 5.0
- link leg_fr: mass 0.4 -> 5.0
Joints:
- joint hip_bl: limit effort=60 velocity=6.0 -> lower=-0.6 upper=0.6 effort=60 velocity=6.0
- joint hip_br: limit effort=60 velocity=6.0 -> lower=-0.6 upper=0.6 effort=60 velocity=6.0
- joint hip_fl: limit effort=60 velocity=6.0 -> lower=-0.6 upper=0.6 effort=60 velocity=6.0
- joint hip_fr: limit effort=60 velocity=6.0 -> lower=-0.6 upper=0.6 effort=60 velocity=6.0
